File: mcu.kicad_sch (KiCad schematic)
At the start: 25 parts, among them U1 W25Q32JVSS, U2 RP2040, Y1 12M 18pF

Commit message: v2: ADV7513 and FFC
Large work much progress - almost routed
Parts:
- added J7: Misc, Connector_PinHeader_2.00mm:PinHeader_2x04_P2.00mm_Vertical, symbol Connector_Generic:Conn_02x04_Odd_Even
Connections:
- net CFG_SW3 is gone; now on net MCU_VID_SCL: U2.32 (GPIO21)
- net CFG_SW4 is gone; now on net MCU_VID_SDA: U2.31 (GPIO20)
- net +3V3: now also J7.2 (Pin_2)
- net GND: now also J7.4 (Pin_4), J7.8 (Pin_8)
- net MCU_VID_SCL: no longer U2.41 (GPIO29_ADC3)
- net MCU_VID_SDA: no longer U2.40 (GPIO28_ADC2)
- net CFG_SW1 renamed spare27
- net spare27: now also J7.1 (Pin_1)
- net CFG_SW2 renamed spare26
- net spare26: now also J7.3 (Pin_3)
- net MCU_A1 renamed spare24
- net spare24: now also J7.7 (Pin_7)
- net MCU_A2 renamed spare25
- net spare25: now also J7.5 (Pin_5)
- new net ID_DET: U2.41 (GPIO29_ADC3)
- new net spare28: J7.6 (Pin_6), U2.40 (GPIO28_ADC2)
Other:
- note added: "ID_DET identifies the interposer/adapter board, e.g. to choose a different bitstream"
- note added: "Make 20/21 SDA/SCL? which order?"
- note added: "Misc header: - Cfg links if needed - I2S DAC if needed!"
- moved on the sheet: C2, C4

Commit message: 2.0 candiate: routed, looks neat, passes DRC
DVI differential pairs aren't tuned that nicely, but 'probs ok'
Parts:
- J7: footprint Connector_PinHeader_2.00mm:PinHeader_2x04_P2.00mm_Vertical -> Connector_PinHeader_2.54mm:PinHeader_2x04_P2.54mm_Vertical
Connections:
- net FPGA_CLK: now also U2.36 (GPIO24); no longer U2.35 (GPIO23)
- net MCU_VID_IRQ: now also U2.32 (GPIO21); no longer U2.34 (GPIO22)
- net MCU_VID_SCL: now also U2.35 (GPIO23); no longer U2.32 (GPIO21)
- net MCU_VID_SDA: now also U2.34 (GPIO22); no longer U2.31 (GPIO20)
- net spare24: no longer names the net of J7.7 (Pin_7)
- net spare24: no longer U2.36 (GPIO24)
- new net VID_I2S_MCLK: U2.31 (GPIO20)
Other:
- note removed: "Make 20/21 SDA/SCL? which order?"
Changed lines of the file:
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@@
-    (stroke (width 0) (type default) (color 0 0 0 0))
-  )
-  (wire (pts (xy 25.4 140.97) (xy 34.29 140.97))
     (stroke (width 0) (type default) (color 0 0 0 0))
   )
@@
     (effects (font (size 1.27 1.27)) (justify left bottom))
   )
-  (text "Make 20/21 SDA/SCL?  which order?" (at 203.2 142.24 0)
-    (effects (font (size 1.27 1.27)) (justify left bottom))
-  )
   (text "E.g. ABL-12.000MHZ-B2" (at 67.31 101.6 0)
     (effects (font (size 1.27 1.27)) (justify left bottom))
@@
     (effects (font (size 1.27 1.27)) (justify left bottom))
   )
-  (label "spare24" (at 209.55 121.92 0)
-    (effects (font (size 1.27 1.27)) (justify left bottom))
-  )
   (label "spare25" (at 25.4 138.43 0)
     (effects (font (size 1.27 1.27)) (justify left bottom))
@@
     (effects (font (size 1.27 1.27)) (justify left bottom))
   )
-  (label "V_SCL" (at 198.12 114.3 0)
+  (label "V_SCL" (at 198.12 119.38 0)
     (effects (font (size 1.27 1.27)) (justify left bottom))
   )
@@
     (effects (font (size 1.27 1.27)) (justify left bottom))
   )
-  (label "spare24" (at 25.4 140.97 0)
-    (effects (font (size 1.27 1.27)) (justify left bottom))
-  )
   (label "V_SDA" (at 260.35 34.29 0)
     (effects (font (size 1.27 1.27)) (justify left bottom))
@@
     (effects (font (size 1.27 1.27)) (justify left bottom))
   )
-  (label "V_SDA" (at 198.12 111.76 0)
+  (label "V_SDA" (at 198.12 116.84 0)
     (effects (font (size 1.27 1.27)) (justify left bottom))
   )
@@
     )
   )
-  (global_label "MCU_VID_IRQ" (shape input) (at 209.55 116.84 0) (fields_autoplaced)
-    (effects (font (size 1.27 1.27)) (justify left))
-    (property "Intersheet References" "${INTERSHEET_REFS}" (id 0) (at 224.1188 116.7606 0)
+  (global_label "MCU_VID_IRQ" (shape input) (at 209.55 114.3 0) (fields_autoplaced)
+    (effects (font (size 1.27 1.27)) (justify left))
+    (property "Intersheet References" "${INTERSHEET_REFS}" (id 0) (at 224.1188 114.2206 0)
+      (effects (font (size 1.27 1.27)) (justify left) hide)
+    )
+  )
+  (global_label "VID_I2S_MCLK" (shape output) (at 209.55 111.76 0) (fields_autoplaced)
+    (effects (font (size 1.27 1.27)) (justify left))
+    (property "Intersheet References" "${INTERSHEET_REFS}" (id 0) (at 224.905 111.6806 0)
       (effects (font (size 1.27 1.27)) (justify left) hide)
     )
@@
     )
   )
-  (global_label "FPGA_CLK" (shape output) (at 209.55 119.38 0) (fields_autoplaced)
-    (effects (font (size 1.27 1.27)) (justify left))
-    (property "Intersheet References" "${INTERSHEET_REFS}" (id 0) (at 221.216 119.3006 0)
+  (global_label "FPGA_CLK" (shape output) (at 209.55 121.92 0) (fields_autoplaced)
+    (effects (font (size 1.27 1.27)) (justify left))
+    (property "Intersheet References" "${INTERSHEET_REFS}" (id 0) (at 221.216 121.8406 0)
       (effects (font (size 1.27 1.27)) (justify left) hide)
     )
@@
     )
   )
-  (global_label "MCU_VID_SCL" (shape output) (at 209.55 114.3 0) (fields_autoplaced)
-    (effects (font (size 1.27 1.27)) (justify left))
-    (property "Intersheet References" "${INTERSHEET_REFS}" (id 0) (at 224.4212 114.2206 0)
+  (global_label "MCU_VID_SCL" (shape output) (at 209.55 119.38 0) (fields_autoplaced)
+    (effects (font (size 1.27 1.27)) (justify left))
+    (property "Intersheet References" "${INTERSHEET_REFS}" (id 0) (at 224.4212 119.3006 0)
       (effects (font (size 1.27 1.27)) (justify left) hide)
     )
@@
     )
   )
-  (global_label "MCU_VID_SDA" (shape bidirectional) (at 209.55 111.76 0) (fields_autoplaced)
-    (effects (font (size 1.27 1.27)) (justify left))
-    (property "Intersheet References" "${INTERSHEET_REFS}" (id 0) (at 224.4817 111.6806 0)
+  (global_label "MCU_VID_SDA" (shape bidirectional) (at 209.55 116.84 0) (fields_autoplaced)
+    (effects (font (size 1.27 1.27)) (justify left))
+    (property "Intersheet References" "${INTERSHEET_REFS}" (id 0) (at 224.4817 116.7606 0)
       (effects (font (size 1.27 1.27)) (justify left) hide)
     )
@@
     (property "Reference" "J7" (id 0) (at 40.64 127 0))
     (property "Value" "Misc" (id 1) (at 40.64 129.54 0))
-    (property "Footprint" "Connector_PinHeader_2.00mm:PinHeader_2x04_P2.00mm_Vertical" (id 2) (at 39.37 135.89 0)
-      (effects (font (size 1.27 1.27)) hide)
-    )
+    (property "Footprint" "Connector_PinHeader_2.54mm:PinHeader_2x04_P2.54mm_Vertical" (id 2) (at 39.37 135.89 0)
+      (effects (font (size 1.27 1.27)) hide)
+    )
