File: video.kicad_sch (KiCad schematic)
At the start: 37 parts, among them U4 TDA19988BHN{slash}C1,557, U7 TLV70018_SOT23-5

Commit message: v2: ADV7513 and FFC
Large work much progress - almost routed
Parts:
- removed FB6: FerriteBead_Small, Inductor_SMD:L_0603_1608Metric, symbol Device:FerriteBead_Small
- removed TP6: AP3, TestPoint:TestPoint_Pad_D1.0mm, symbol Connector:TestPoint
- removed U4: TDA19988BHN/C1,557, matt:QFN50P900X900X100-65N, symbol matt:TDA19988BHN{brace}slash}C1,557
- added C58, C59: 0.1u, Capacitor_SMD:C_0603_1608Metric, symbol Device:C
- added D2: ESDA6V1BC6, Package_TO_SOT_SMD:SOT-23-6, symbol Power_Protection:ESDA6V1BC6
- added D3: D, Diode_SMD:D_0603_1608Metric, symbol Device:D
- added D4: RCLAMP3328P, Package_DFN_QFN:UDFN-9_1.0x3.8mm_P0.5mm, symbol Power_Protection:RCLAMP3328P
- added F1: 50mA, Fuse:Fuse_1206_3216Metric_Pad1.42x1.75mm_HandSolder, symbol Device:Fuse
- added J8: HDMI_A, Connector_HDMI:HDMI_A_Molex_208658-1001_Horizontal, symbol Connector:HDMI_A
- added R18, R19: 2K, Resistor_SMD:R_0603_1608Metric, symbol Device:R
- added R20: 27K, Resistor_SMD:R_0603_1608Metric, symbol Device:R
- added R21: 22, Resistor_SMD:R_0603_1608Metric, symbol Device:R
- added U4: ADV7513BSWZ, matt:QFP50P1200X1200X160-65N, symbol matt:ADV7513BSWZ
- C42: value 1u -> 10u
- C44: value 10u -> 0.1u; footprint Capacitor_SMD:C_0805_2012Metric -> Capacitor_SMD:C_0603_1608Metric
- C46, C52: value 1u -> 0.1u
- R12, R13: value 10K -> 2K
- R14: value 10K, 1% -> 887, 1%
- TP5: value AP4 -> SPD
- TP7: value AP2 -> MCLK
Connections:
- net +1V8: no longer C44.1, C46.1, FB7.1
- net +3V3: now also FB7.1, R19.1
- net +5V: now also F1.2
- net ALT_VID_I2S_CLK: now also RN13.2 (R2.1); no longer RN13.1 (R1.1)
- net ALT_VID_I2S_DATA: now also RN13.1 (R1.1); no longer RN13.3 (R3.1)
- net ALT_VID_I2S_WS: now also RN13.3 (R3.1); no longer RN13.2 (R2.1)
- net GND: now also C58.2, C59.2, D2.2 (COM), D2.5 (COM), D4.3 (A), J8.11 (CKS), J8.17 (GND), J8.2 (D2S), J8.5 (D1S), J8.8 (D0S), J8.SH, R18.2, U4.65 (EP)
- net MCU_VID_IRQ: now also R19.2, U4.28 (INT)
- net MCU_VID_SCL: now also U4.35 (SCL)
- net MCU_VID_SDA: now also U4.36 (SDA)
- net RGB0: now also RN4.1 (R1.1); no longer RN5.4 (R4.1)
- net RGB1: now also RN5.4 (R4.1); no longer RN5.3 (R3.1)
- net RGB10: now also RN3.2 (R2.1); no longer RN3.3 (R3.1)
- net RGB11: now also RN3.1 (R1.1); no longer RN3.2 (R2.1)
- net RGB16: now also RN2.4 (R4.1); no longer RN4.1 (R1.1)
- net RGB17: now also RN2.3 (R3.1); no longer RN2.4 (R4.1)
- net RGB18: now also RN2.2 (R2.1); no longer RN2.3 (R3.1)
- net RGB19: now also RN2.1 (R1.1); no longer RN2.2 (R2.1)
- net RGB2: now also RN5.3 (R3.1); no longer RN5.2 (R2.1)
- net RGB20: now also RN1.4 (R4.1); no longer RN2.1 (R1.1)
- net RGB21: now also RN1.3 (R3.1); no longer RN1.4 (R4.1)
- net RGB22: now also RN1.2 (R2.1); no longer RN1.3 (R3.1)
- net RGB23: now also RN1.1 (R1.1); no longer RN1.2 (R2.1)
- net RGB3: now also RN5.2 (R2.1); no longer RN5.1 (R1.1)
- net RGB4: now also RN5.1 (R1.1); no longer RN6.4 (R4.1)
- net RGB5: now also RN6.4 (R4.1); no longer RN6.3 (R3.1)
- net RGB6: now also RN6.3 (R3.1); no longer RN6.2 (R2.1)
- net RGB7: now also RN6.2 (R2.1); no longer RN6.1 (R1.1)
- net RGB8: now also RN6.1 (R1.1); no longer RN1.1 (R1.1)
- net RGB9: now also RN3.3 (R3.1); no longer RN3.4 (R4.1)
- net VID_OUT_HS: now also RN4.3 (R3.1); no longer RN4.4 (R4.1)
- net VID_OUT_PCLK: now also RN3.4 (R4.1); no longer RN3.1 (R1.1)
- net VID_OUT_VS: now also RN4.4 (R4.1); no longer RN4.3 (R3.1)
- net at TP7.1: now also U4.4 (MCLK)
- net at RN13.6 (R3.2): now also RN12.6 (R3.2), U4.10 (LRCLK); no longer RN12.8 (R1.2)
- net at RN13.7 (R2.2): now also RN12.7 (R2.2), U4.9 (SCLK); no longer RN12.6 (R3.2)
- net at RN13.8 (R1.2): now also RN12.8 (R1.2), U4.5 (I2S0); no longer RN12.7 (R2.2)
- net at RN4.5 (R4.2): now also U4.2 (VSYNC)
- net at RN4.6 (R3.2): now also U4.64 (HSYNC)
- net at RN4.7 (R2.2): now also U4.63 (DE)
- net at RN4.8 (R1.2): now also U4.62 (D0)
- net at R14.1: now also U4.14 (R_EXT)
- net at RN7.5 (R4.2): now also U4.48 (D12)
- net at RN7.6 (R3.2): now also U4.47 (D13)
- net at RN7.7 (R2.2): now also U4.46 (D14)
- net at RN7.8 (R1.2): now also U4.45 (D15)
- net at RN1.7 (R2.2): now also U4.38 (D22)
- net at RN1.6 (R3.2): now also U4.39 (D21)
- net at RN1.5 (R4.2): now also U4.40 (D20)
- net at RN2.8 (R1.2): now also U4.41 (D19)
- net at RN2.7 (R2.2): now also U4.42 (D18)
- net at RN2.6 (R3.2): now also U4.43 (D17)
- net at RN2.5 (R4.2): now also U4.44 (D16)
- net at TP5.1: now also U4.3 (SPDIF)
- net at RN6.8 (R1.2): now also U4.54 (D8)
- net at RN6.7 (R2.2): now also U4.55 (D7)
- net at RN6.6 (R3.2): now also U4.56 (D6)
- net at RN6.5 (R4.2): now also U4.57 (D5)
- net at RN3.7 (R2.2): now also U4.50 (D10)
- net at RN5.8 (R1.2): now also U4.58 (D4)
- net at RN5.7 (R2.2): now also U4.59 (D3)
- net at RN5.6 (R3.2): now also U4.60 (D2)
- net at RN5.5 (R4.2): now also U4.61 (D1)
- net at RN3.6 (R3.2): now also U4.52 (D9)
- net at RN3.5 (R4.2): now also U4.53 (CLK)
- net at RN1.8 (R1.2): now also U4.37 (D23)
- net PCLK_R: no longer names the net of RN3.8 (R1.2)
- net PCLK_R: now also U4.49 (D11)
- net VDDA renamed AVDD
- net AVDD: now also C44.1, C46.1, U4.15 (AVDD), U4.19 (AVDD), U4.25 (AVDD)
- net VDDA_PLL renamed DVDD
- net DVDD: now also C53.1, C58.1, C59.1, U4.1 (DVDD), U4.11 (DVDD), U4.31 (DVDD), U4.51 (DVDD)
- net VDDA_TX renamed PVDD
- net PVDD: now also C52.1, U4.12 (PVDD), U4.13 (BGVDD)
- removed net VDD_CORE: C52.1, C53.1
- net VDD_IO renamed DVDD3
- net DVDD3: now also R20.1, U4.29 (DVDD_3V)
- net VID_DISP_SCL renamed DDC_SCL
- net DDC_SCL: now also D2.3 (TVS2), J8.15 (SCL), U4.33 (DDCSCL)
- net VID_DISP_SDA renamed DDC_SDA
- net DDC_SDA: now also D2.4 (TVS3), J8.16 (SDA), U4.34 (DDCSDA)
- new net: D3.2 (A), R20.2
- new net: R18.1, U4.22 (PD)
- new net: R21.2, U4.32 (CEC_CLK)
- new net CEC: D2.6 (TVS4), D3.1 (K), J8.13 (CEC), U4.30 (CEC)
- new net HDMI5V: F1.1, J8.18 (+5V)
- new net HPD: D2.1 (TVS1), J8.19 (HPD), U4.16 (HPD)
- new net TX0+: D4.7 (K6), J8.7 (D0+), U4.21 (TX0+)
- new net TX0-: D4.4 (K3), J8.9 (D0-), U4.20 (TX0−)
- new net TX1+: D4.2 (K2), J8.4 (D1+), U4.24 (TX1+)
- new net TX1-: D4.8 (K7), J8.6 (D1-), U4.23 (TX1−)
- new net TX2+: D4.1 (K1), J8.1 (D2+), U4.27 (TX2+)
- new net TX2-: D4.9 (K8), J8.3 (D2-), U4.26 (TX2−)
- new net TXC+: D4.6 (K5), J8.10 (CK+), U4.18 (TXC+)
- new net TXC-: D4.5 (K4), J8.12 (CK-), U4.17 (TXC−)
- new net VID_CEC_CLK: R21.1
Other:
- note added: "ADV7513 DS says MCLK isn't needed. Adding a TP in case a bodge is necessary!"
- note added: "ESD protection"
- note added: "Ir < 1.5uA C < 6pF"
- note added: "NC"
- note added: "Or similar, e.g. SP7538PUTG"
- note added: "Supposed to use 10uH filter"
- note removed: "DNF pullups?"
- note removed: "FIXME: ESD protection pls"
- note removed: "TDA19988 consumes ~100mA on 1.8V rail(s)"
- moved on the sheet: C42, C43, C45, C47, C48, C50, C54, C56, FB3, FB4, FB5, FB7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

Commit message: 2.0 candiate: routed, looks neat, passes DRC
DVI differential pairs aren't tuned that nicely, but 'probs ok'
Parts:
- removed TP7: MCLK, TestPoint:TestPoint_Pad_D1.0mm, symbol Connector:TestPoint
Connections:
- net ALT_VID_I2S_CLK: now also RN13.3 (R3.1); no longer RN13.2 (R2.1)
- net ALT_VID_I2S_DATA: now also RN13.2 (R2.1); no longer RN13.1 (R1.1)
- net ALT_VID_I2S_WS: now also RN13.4 (R4.1); no longer RN13.3 (R3.1)
- net DDC_SCL: now also D2.4 (TVS3); no longer D2.3 (TVS2)
- net DDC_SDA: now also D2.3 (TVS2); no longer D2.4 (TVS3)
- net VID_I2S_CLK: now also RN12.3 (R3.1); no longer RN12.2 (R2.1)
- net VID_I2S_DATA: now also RN12.2 (R2.1); no longer RN12.1 (R1.1)
- net VID_I2S_WS: now also RN12.4 (R4.1); no longer RN12.3 (R3.1)
- net at U4.4 (MCLK): now also RN12.8 (R1.2), RN13.8 (R1.2)
- net at RN13.5 (R4.2): now also RN12.5 (R4.2), U4.10 (LRCLK)
- net at RN12.6 (R3.2), RN13.6 (R3.2): now also U4.9 (SCLK); no longer U4.10 (LRCLK)
- net at RN12.7 (R2.2), RN13.7 (R2.2): now also U4.5 (I2S0); no longer U4.9 (SCLK)
- new net ALT_VID_I2S_MCLK: RN13.1 (R1.1)
- new net VID_I2S_MCLK: RN12.1 (R1.1)
