File: arc-dvi.kicad_pcb (KiCad board)
At the start: 4 copper layers, 100 x 77 mm, 143 parts, among them J1 Connector_50pin_FFC, J2 5V_IN, J3 SWD, J4 BOOT, J5 USB_B_Micro, J6 PWR_USB, J7 Misc, J8 HDMI_A, Q1 Q_NPN_BCE, U1 W25Q32JVSS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

Commit message: Updated date, made board narrower, added dims
Parts:
- moved U5 2.50 mm to (64.0, 86.5)
- moved C34 2.50 mm to (58.8, 97.2)
- moved C35 2.50 mm to (58.3, 88.2)
- moved C36 2.50 mm to (62.2, 92.8)
- moved C37 2.50 mm to (65.8, 92.8)
- moved C38 2.50 mm to (69.8, 88.2)
- moved FB1 2.50 mm to (63.8, 98.5)
- moved J2 2.50 mm to (62.0, 103.0)
- moved TP1 2.50 mm to (58.2, 79.0)
- moved TP2 2.50 mm to (69.5, 79.0)
- moved TP8 2.50 mm to (64.0, 79.0)
- moved G*** 1.06 mm to (131.5, 102.5)
Routing:
- net GND: track 963.1 -> 960.4 mm
- net +5V: track 167.1 -> 168.3 mm
- net +3V3: track 468.3 -> 469.5 mm
Other:
- board size 100 x 77 mm -> 92.5 x 77 mm
- board text added: "v2.0 220523 (c) 2023 Matt Evans"
- board text removed: "v2.0 210523 (c) 2023 Matt Evans"

Commit message: Made board slightly smaller, re-centered contact point, tidied
Good to go, DRC clean.
Parts:
- moved TP21 8.49 mm to (136.0, 66.8)
- moved TP19 7.06 mm to (116.5, 120.5)
- moved F1 5.34 mm to (132.2, 57.2), turned to 90 degrees
- moved J2 5.25 mm to (65.4, 107.0), turned to 180 degrees
- moved H2 5.00 mm to (140.0, 117.1)
- moved H4 5.00 mm to (60.0, 117.1)
- moved TP4 3.04 mm to (98.5, 120.5)
- moved R17 3.01 mm to (105.8, 72.2), turned to 0 degrees
- moved TP3 3.00 mm to (133.6, 115.2)
- moved TP20 2.86 mm to (133.6, 111.0)
- moved TP6 2.51 mm to (96.8, 116.0)
- moved J1 2.50 mm to (80.0, 119.5)
- moved C39 2.02 mm to (111.2, 118.7)
- moved C40 2.02 mm to (102.4, 120.9)
- moved C41 2.02 mm to (101.7, 118.3)
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Routing:
- net +5V: track 168.3 -> 176.3 mm
- net Net-(FB1-Pad2): track 4.16 -> 10.9 mm
- net /Video/HDMI5V: track 13.1 -> 16.9 mm
- net +3V3: track 469.5 -> 472.3 mm
- net VnVCS: track 14.8 -> 12.3 mm
- net VD31: track 14.8 -> 12.3 mm
- net VFLYBK: track 14.5 -> 12.0 mm
- net VD11: track 33.0 -> 30.5 mm
- net VCKIN: track 14.5 -> 12.0 mm
- net VD28: track 18.0 -> 15.5 mm
- net VnVIDW: track 14.8 -> 12.3 mm
- net VnVIDRQ: track 14.5 -> 12.0 mm
- net VnSNDRQ: track 14.5 -> 12.0 mm
- net VnHS: track 14.8 -> 12.3 mm
- net VVIDAK: track 14.5 -> 12.0 mm
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Other:
- board size 92.5 x 77 mm -> 92.5 x 74 mm
- board text added: "(c) 2023 Matt Evans"
- board text added: "5V"
- board text added: "v2.0 010623"
- board text removed: "50"
- board text removed: "Gnd 5V"
- board text removed: "v2.0 220523 (c) 2023 Matt Evans"

Commit message: Add README, licence
Other:
- board text added: "Revision 2.0 Copyright 2023 Matt Evans CC BY-NC-SA 3.0"
Changed lines of the file:
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@@
     (effects (font (size 1 1) (thickness 0.15)))
+  )
+  (gr_text "Revision 2.0\n\nCopyright 2023 Matt Evans\nCC BY-NC-SA 3.0" (at 178.25 170.5) (layer "Cmts.User")
+    (effects (font (size 1 1) (thickness 0.15)) (justify left))
   )
   (dimension (type aligned) (layer "Dwgs.User")
