File: arc-dvi.kicad_sch (KiCad schematic)
At the start: 26 parts, among them J1 Conn_01x24_MountingPin, J2 VIDC Interposer, J3 SWD, J4 BOOT, J5 USB_B_Micro, J6 PWR, U5 LT1963AxST-3.3

Commit message: v2: ADV7513 and FFC
Large work much progress - almost routed
Parts:
- removed J1: Conn_01x24_MountingPin, Connector_FFC-FPC:TE_2-1734839-4_1x24-1MP_P0.5mm_Horizontal, symbol Connector_Generic_MountingPin:Conn_01x24_MountingPin
- removed J2: VIDC Interposer, Connector_PinHeader_2.54mm:PinHeader_2x25_P2.54mm_Vertical, symbol matt:Connector_50pin
- removed J6: PWR, Connector_PinHeader_2.54mm:PinHeader_1x03_P2.54mm_Vertical, symbol Connector:Conn_01x03_Male
- added J1: Connector_50pin_FFC, Connector_FFC-FPC:Hirose_FH12-50S-0.5SH_1x50-1MP_P0.50mm_Horizontal, symbol matt:Connector_50pin_FFC
- added J2: 5V_IN, Connector_PinHeader_2.54mm:PinHeader_1x02_P2.54mm_Horizontal, symbol Connector:Conn_01x02_Male
- added J6: PWR_USB, Connector_PinHeader_2.54mm:PinHeader_1x02_P2.54mm_Vertical, symbol Connector:Conn_01x02_Male
- added TP6: P50, TestPoint:TestPoint_Pad_D1.0mm, symbol Connector:TestPoint
Connections:
- net +5V: now also J6.1 (Pin_1)
- net GND: now also J1.16, J1.24, J1.32, J1.40, J1.47, J1.8, J1.MP, J2.2 (Pin_2)
- net VBUS: now also J6.2 (Pin_2)
- net VCKIN: now also J1.44
- net VD0: now also J1.1
- net VD1: now also J1.2
- net VD10: now also J1.12
- net VD11: now also J1.13
- net VD12: now also J1.14
- net VD13: now also J1.15
- net VD14: now also J1.17
- net VD15: now also J1.18
- net VD16: now also J1.19
- net VD17: now also J1.20
- net VD18: now also J1.21
- net VD19: now also J1.22
- net VD2: now also J1.3
- net VD20: now also J1.23
- net VD21: now also J1.25
- net VD22: now also J1.26
- net VD23: now also J1.27
- net VD24: now also J1.28
- net VD25: now also J1.29
- net VD26: now also J1.30
- net VD27: now also J1.31
- net VD28: now also J1.33
- net VD29: now also J1.34
- net VD3: now also J1.4
- net VD30: now also J1.35
- net VD31: now also J1.36
- net VD4: now also J1.5
- net VD5: now also J1.6
- net VD6: now also J1.7
- net VD7: now also J1.9
- net VD8: now also J1.10
- net VD9: now also J1.11
- net VFLYBK: now also J1.43
- net VSNDAK: now also J1.46
- net VVIDAK: now also J1.45
- net VnHS: now also J1.38
- net VnSNDRQ: now also J1.42
- net VnVCS: now also J1.39
- net VnVIDRQ: now also J1.41
- net VnVIDW: now also J1.37
- net HOST_5V: no longer names the net of FB1.2
- net HOST_5V: now also J2.1 (Pin_1)
- new net: J1.50, TP6.1
- new net ID_DET: J1.49
Other:
- note added: "Development link, to power board from USB 5V"
- note added: "FFC 50-pin 0.5mm connector: Same orientation on all boards: use FLIPPED cable"
- note added: "Main power input"
- note added: "pin 50 possible future 5V for hacks, TP"
- note removed: "A to MCU"
- note removed: "External power, and link enabling VBUS to power board"
- note removed: "FFC to SocketBoard"
- note removed: "NOTE: Pins are reversed with respect to the same connector on the SocketBrd, e.g. HPD is on the far left (RHS looking at back of connector). Thus, FPC NON-FLIPPED (same side) cable should be used."
- note removed: "Switches to MCU"
- moved on the sheet: C57, FB1, J3, J4, R15

Commit message: 2.0 candiate: routed, looks neat, passes DRC
DVI differential pairs aren't tuned that nicely, but 'probs ok'
Parts:
- added H5: MountingHole, MountingHole:MountingHole_3.2mm_M3, symbol Mechanical:MountingHole
Changed lines of the file:
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@@
     (pin "1")
+  )
+  (symbol (lib_id "Mechanical:MountingHole") (at 141.605 255.27 0) (unit 1)
+    (in_bom yes) (on_board yes) (fields_autoplaced)
+    (property "Reference" "H5" (id 0) (at 144.145 253.9999 0)
+      (effects (font (size 1.27 1.27)) (justify left))
+    )
+    (property "Value" "MountingHole" (id 1) (at 144.145 256.5399 0)
+      (effects (font (size 1.27 1.27)) (justify left))
+    )
+    (property "Footprint" "MountingHole:MountingHole_3.2mm_M3" (id 2) (at 141.605 255.27 0)
+      (effects (font (size 1.27 1.27)) hide)
+    )
+    (property "Datasheet" "~" (id 3) (at 141.605 255.27 0)
+      (effects (font (size 1.27 1.27)) hide)
+    )
   )
   (symbol (lib_id "Device:C_Polarized") (at 262.89 154.94 0) (unit 1)
@@
       (reference "H4") (unit 1) (value "MountingHole") (footprint "MountingHole:MountingHole_3.2mm_M3")
     )
+    (path "/2860f837-5cb0-411f-807f-4fe07e12b841"
+      (reference "H5") (unit 1) (value "MountingHole") (footprint "MountingHole:MountingHole_3.2mm_M3")
+    )
     (path "/2fda9f65-cd41-4a12-bfe6-6ae3ba001749"
       (reference "J1") (unit 1) (value "Connector_50pin_FFC") (footprint "Connector_FFC-FPC:Hirose_FH12-50S-0.5SH_1x50-1MP_P0.50mm_Horizontal")
@@
     )
     (path "/39ecbee3-68dc-4e5f-bbac-36474508dffd/7f799f42-1a4d-4f3b-9c9a-0430320c0d7c"
-      (reference "J7") (unit 1) (value "Misc") (footprint "Connector_PinHeader_2.00mm:PinHeader_2x04_P2.00mm_Vertical")
+      (reference "J7") (unit 1) (value "Misc") (footprint "Connector_PinHeader_2.54mm:PinHeader_2x04_P2.54mm_Vertical")
     )
     (path "/adf79454-fa21-4ca1-b75b-79de44e40f87/cad20d73-ab30-4c2f-8632-1673c10eded7"
@@
       (reference "TP6") (unit 1) (value "P50") (footprint "TestPoint:TestPoint_Pad_D1.0mm")
     )
-    (path "/adf79454-fa21-4ca1-b75b-79de44e40f87/3f89818b-d890-49e2-a916-38449ebc09bd"
-      (reference "TP7") (unit 1) (value "MCLK") (footprint "TestPoint:TestPoint_Pad_D1.0mm")
-    )
     (path "/f778a554-bb14-4f45-878c-7eddbb5c99c6"
       (reference "TP8") (unit 1) (value "Gnd") (footprint "TestPoint:TestPoint_Pad_1.5x1.5mm")
@@
       (reference "TP14") (unit 1) (value "217") (footprint "TestPoint:TestPoint_Pad_D1.0mm")
     )
-    (path "/838b72cc-eb9e-4020-adeb-4d1da7258fcf/fce2df0a-e3c6-4a82-894e-fe607f55409f"
-      (reference "TP15") (unit 1) (value "219") (footprint "TestPoint:TestPoint_Pad_D1.0mm")
-    )
     (path "/838b72cc-eb9e-4020-adeb-4d1da7258fcf/539a7b65-9154-4554-9522-c93a7666ee4e"

Commit message: Add README, licence
Other:
- note added: "Copyright 2023 Matt Evans CC BY-NC-SA 3.0"
Changed lines of the file:
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@@
+    (effects (font (size 1.27 1.27)) (justify left bottom))
+  )
+  (text "Copyright 2023 Matt Evans\nCC BY-NC-SA 3.0" (at 300.99 266.7 0)
     (effects (font (size 1.27 1.27)) (justify left bottom))
   )
